File: tp_abbate/ESP32.sch (KiCad schematic (older format))
At the start: 20 parts, among them J201 U.FL-R-SMT-1(10), J202 Conn_01x06, J203 Conn_01x12, J204 Conn_01x12, Q201 AO3401A, Q202 2N7002DW, SW201 SW_Push, SW202 SW_Push, U201 ESP32-WROOM-32, U202 Ai-Thinker-Ra-01

Commit message: WIP revisión PCB
Parts:
- removed J202: Conn_01x06, Connector_PinHeader_2.54mm:PinHeader_1x06_P2.54mm_Vertical, symbol Connector_Generic:Conn_01x06
- added J202: Conn_01x04, Connector_PinHeader_2.54mm:PinHeader_1x04_P2.54mm_Vertical, symbol Connector_Generic:Conn_01x04
Connections:
- net GPIO12: now also J203.6 (Pin_6); no longer J203.9 (Pin_9)
- net GPIO13: now also J203.9 (Pin_9); no longer J203.8 (Pin_8)
- net GPIO15: now also J203.8 (Pin_8); no longer J203.7 (Pin_7)
- net GPIO2: now also J203.7 (Pin_7); no longer J203.6 (Pin_6)
- net at U202.5 (DIO0): now also J202.1 (Pin_1)
- net at U202.6 (DIO1): now also J202.2 (Pin_2)
- net at U202.7 (DIO2): now also J202.3 (Pin_3)
- net at U202.8 (DIO3): now also J202.4 (Pin_4)
- no-connect marks 6 -> 8
Changed lines of the file:
@@
 Text Label 8900 3150 0    50   ~ 0
 GPIO16
-Text Label 8900 3550 0    50   ~ 0
+Text Label 8900 3650 0    50   ~ 0
 GPIO15
-Text Label 8900 3650 0    50   ~ 0
+Text Label 8900 3750 0    50   ~ 0
 GPIO13
-Text Label 8900 3750 0    50   ~ 0
+Text Label 8900 3450 0    50   ~ 0
 GPIO12
 Text Label 8900 3250 0    50   ~ 0
 GPIO4
-Text Label 8900 3450 0    50   ~ 0
+Text Label 8900 3550 0    50   ~ 0
 GPIO2
 Text Label 8900 3350 0    50   ~ 0
 GPIO0
-$Comp
-L Connector_Generic:Conn_01x06 J?
-U 1 1 5EF01CF2
-P 9500 2300
-AR Path="/5EF01CF2" Ref="J?"  Part="1"
-AR Path="/5EED5E8D/5EF01CF2" Ref="J202"  Part="1"
-F 0 "J202" H 9580 2292 50  0000 L CNN
-F 1 "Conn_01x06" H 9580 2201 50  0000 L CNN
-F 2 "Connector_PinHeader_2.54mm:PinHeader_1x06_P2.54mm_Vertical" H 9500 2300 50  0001 C CNN
-F 3 "~" H 9500 2300 50  0001 C CNN
-	1    9500 2300
-	1    0    0    -1
-$EndComp
 $Comp
 L power:+3.3V #PWR?
@@
 Wire Wire Line
 	8100 1550 8100 1500
-Wire Wire Line
-	8600 2600 9300 2600
-Wire Wire Line
-	8600 2500 9300 2500
 $Comp
 L tp_abbate:Ai-Thinker-Ra-01 U?
@@
 Wire Wire Line
 	5800 1750 6500 1750
+Entry Wire Line
+	8700 5550 8800 5650
+Entry Wire Line
+	8700 5450 8800 5550
+$Comp
+L Connector_Generic:Conn_01x04 J202
+U 1 1 5EF6E39D
+P 9500 2200
+F 0 "J202" H 9580 2192 50  0000 L CNN
+F 1 "Conn_01x04" H 9580 2101 50  0000 L CNN
+F 2 "Connector_PinHeader_2.54mm:PinHeader_1x04_P2.54mm_Vertical" H 9500 2200 50  0001 C CNN
+F 3 "~" H 9500 2200 50  0001 C CNN
+	1    9500 2200
+	1    0    0    -1
+$EndComp
+NoConn ~ 8600 2600
+NoConn ~ 8600 2500
 Wire Bus Line
 	6400 3750 6400 4450
@@
 Wire Bus Line
 	6400 2750 6400 3650
-Entry Wire Line
-	8700 5550 8800 5650
-Entry Wire Line
-	8700 5450 8800 5550
 $EndSCHEMATC

Commit message: Subo PCB para revisión compañero
Parts:
- renumbered C202 to C10, C203 to C11, C204 to C12, C205 to C13, C201 to C9, J201 to J3, J202 to J4, J203 to J5, J204 to J6, Q201 to Q2, Q202 to Q3, R203 to R10, R204 to R11, R205 to R12, R201 to R8, R202 to R9, SW201 to SW1, SW202 to SW2, U201 to U4, U202 to U5
Other:
- note added: "Close to U4\nVDD pin\n"
- note added: "Close to U5\n3v3 pin\n"
- note removed: "Close to U201\nVDD pin\n"
- note removed: "Close to U202\n3v3 pin\n"

Commit message: Corrijo indicaciones de compañero
Parts:
- J3: footprint U.FL:HRS_U.FL-R-SMT-1(10) -> tp_abbate:HRS_U.FL-R-SMT-1(10)
Changed lines of the file:
@@
 F 0 "J3" H 9100 1950 50  0000 L CNN
 F 1 "U.FL-R-SMT-1(10)" H 9100 1850 50  0000 L CNN
-F 2 "U.FL:HRS_U.FL-R-SMT-1(10)" H 9150 1650 50  0001 L BNN
+F 2 "tp_abbate:HRS_U.FL-R-SMT-1(10)" H 9150 1650 50  0001 L BNN
 F 3 "" H 9150 1650 50  0001 L BNN
 F 4 "U.FL Series 6 Ghz 50 Ohm Ultra-small SMT Coaxial Cable Receptacle" H 9150 1650 50  0001 L BNN "Desc"

Commit message: Revisión Final - Entrega
Other:
- note added: "Close to U5\npin N°1"
- note removed: "Close to\nboard edge"
Changed lines of the file:
@@
 Text Notes 9850 3600 0    100  ~ 20
 GPIOs Headers
-Text Notes 9300 1750 0    50   ~ 0
-Close to\nboard edge
 Wire Wire Line
 	8900 1750 9050 1750
@@
 Wire Bus Line
 	6400 2750 6400 3650
+Text Notes 9300 1750 0    50   ~ 0
+Close to U5\npin N°1
 $EndSCHEMATC
