File: tp_abbate/tp_abbate.kicad_pcb (KiCad board)
At the start: 2 copper layers, 43 x 61.5 mm, 45 parts, among them J101 USB_B_Micro, J102 S2B-PH-K-S, J201 U.FL-R-SMT-1(10), J202 Conn_01x06, J203 Conn_01x12, J204 Conn_01x12, Q101 AO3401A, Q201 AO3401A, Q202 2N7002DW, SW201 SW_Push, SW202 SW_Push, U101 LTC4054ES5-4.2, U102 CP2102-GM-QFN28, U103 MIC5219-3.3YMM, U201 ESP32-WROOM-32, U202 Ai-Thinker-Ra-01

Commit message: WIP revisión PCB
Parts:
- added FID1: Fiducial, Fiducial:Fiducial_0.5mm_Mask1.5mm, F.Cu at (89.0, 118.5)
- added FID2: Fiducial, Fiducial:Fiducial_0.5mm_Mask1.5mm, F.Cu at (100.5, 80.5)
- added FID3: Fiducial, Fiducial:Fiducial_0.5mm_Mask1.5mm, F.Cu at (146.0, 115.0)
- J202: value Conn_01x06 -> Conn_01x04; footprint Connector_PinHeader_2.54mm:PinHeader_1x06_P2.54mm_Vertical -> Connector_PinHeader_2.54mm:PinHeader_1x04_P2.54mm_Vertical
- moved J102 159.1 mm to (92.5, 81.0), turned to 180 degrees
- moved SW201 155.6 mm to (93.0, 84.5), turned to 0 degrees
- moved D102 153.8 mm to (91.0, 90.0), turned to 270 degrees
- moved D103 150.2 mm to (94.0, 90.0), turned to 270 degrees
- moved J101 150.1 mm to (89.0, 99.0), turned to 270 degrees
- moved C106 146.6 mm to (97.0, 90.0), turned to 90 degrees
- moved F101 146.5 mm to (94.0, 95.0), turned to 270 degrees
- moved U103 143.4 mm to (101.5, 87.5), turned to 90 degrees
- moved R106 142.9 mm to (97.0, 95.0), turned to 90 degrees
- moved C102 141.5 mm to (91.5, 108.0), turned to 90 degrees
- moved R103 140.1 mm to (95.5, 99.5), turned to 180 degrees
- moved C108 138.8 mm to (105.5, 87.5), turned to 90 degrees
- moved R102 138.7 mm to (95.5, 102.5), turned to 180 degrees
- moved Q101 138.6 mm to (101.5, 93.5), turned to 90 degrees
- moved C103 138.3 mm to (94.0, 108.0), turned to 90 degrees
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Connections:
- J203 pad 6: /ESP32/GPIO2 -> /ESP32/GPIO12
- J203 pad 7: /ESP32/GPIO15 -> /ESP32/GPIO2
- J203 pad 8: /ESP32/GPIO13 -> /ESP32/GPIO15
- J203 pad 9: /ESP32/GPIO12 -> /ESP32/GPIO13
- U202 pad 10: Net-(J202-Pad5) -> Net-(U202-Pad10)
- U202 pad 11: Net-(J202-Pad6) -> Net-(U202-Pad11)
Routing:
- net +3V3: track 0.00 -> 124.0 mm, vias 0 -> 3
- net GND: track 0.00 -> 119.3 mm, vias 0 -> 18
- net +5V: track 0.00 -> 110.7 mm, vias 0 -> 2
- net /ESP32/CHIP_PU: track 0.00 -> 90.8 mm, vias 0 -> 5
- net /ESP32/GPIO0: track 0.00 -> 65.3 mm, vias 0 -> 2
- net +BATT: track 0.00 -> 43.7 mm, vias 0 -> 3
- net /ESP32/GPIO12: track 0.00 -> 42.7 mm, vias 0 -> 2
- net /ESP32/GPIO21: track 0.00 -> 42.0 mm, vias 0 -> 2
- net /ESP_RXD: track 0.00 -> 37.4 mm, vias 0 -> 2
- net /ESP_TXD: track 0.00 -> 37.0 mm, vias 0 -> 2
- net /ESP32/GPIO22: track 0.00 -> 35.5 mm, vias 0 -> 1
- net /ESP32/GPIO13: track 0.00 -> 34.9 mm, vias 0 -> 2
- net /ESP32/LORA_SS: track 0.00 -> 34.1 mm, vias 0 -> 1
- net /ESP32/LORA_MISO: track 0.00 -> 33.1 mm, vias 0 -> 1
- net /ESP32/LORA_SCK: track 0.00 -> 32.7 mm, vias 0 -> 1
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- added copper zone on B.Cu, net GND
Other:
- board size 43 x 61.5 mm -> 62 x 43 mm
- net class Default: via_dia 1.27 -> 1; via_drill 0.7 -> 0.5
- net class USB_Conn: via_dia 1.27 -> 1; via_drill 0.7 -> 0.5
- rule pad_to_mask_clearance: 0.05 -> 0.1
- board text added: "Grillas: - Principal 0,5mm - Alternativa 0,25mm Separación al borde: 0,5mm Estándar de fabricación: http://www.mayerpcb.com/uploads/estandares.pdf Net class "Default" : Mayer 10 mils - Ancho mínimo de traza 0,25mm - Separacion mínima entre trazas 0,25mm - Diametro mínimo de via 1mm - Perforación mínima de via 0,5m Net class "USB_Conn" : Mayer 8 mils - Ancho mínimo de traza 0,2mm - Separacion míni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"
- board text added: "Reglas de diseño y fabricación"

Commit message: Subo PCB para revisión compañero
Parts:
- removed C106: 2.2uF, Capacitor_Tantalum_SMD:CP_EIA-3216-18_Kemet-A_Pad1.58x1.35mm_HandSolder
- removed D101: LED_YELLOW, LED_SMD:LED_0805_2012Metric_Pad1.15x1.40mm_HandSolder
- removed F101: 5V 500mA, Fuse:Fuse_0603_1608Metric_Pad1.05x0.95mm_HandSolder
- removed U103: MIC5219-3.3YMM, Package_SO:MSOP-8_3x3mm_P0.65mm
- removed U201: ESP32-WROOM-32, RF_Module:ESP32-WROOM-32
- added C6: 2.2uF, Capacitor_Tantalum_SMD:CP_EIA-3216-18_Kemet-A_Pad1.58x1.35mm_HandSolder, F.Cu at (97.0, 90.0)
- added D1: LED_YELLOW, LED_SMD:LED_0805_2012Metric_Pad1.15x1.40mm_HandSolder, F.Cu at (109.0, 102.0)
- added F1: 5V 500mA, Fuse:Fuse_0603_1608Metric_Pad1.05x0.95mm_HandSolder, F.Cu at (94.0, 95.0)
- added U3: MIC5219-3.3YMM, Package_SO:MSOP-8_3x3mm_P0.65mm, F.Cu at (101.5, 87.5)
- added U4: ESP32-WROOM-32, RF_Module:ESP32-WROOM-32, F.Cu at (132.0, 99.5)
- moved D2 0.25 mm to (90.8, 90.0)
- renumbered C101 to C1, C202 to C10, C203 to C11, C204 to C12, C205 to C13, C102 to C2, C103 to C3, C104 to C4, C105 to C5, C107 to C7, C108 to C8, C201 to C9, D102 to D2, D103 to D3, J101 to J1, J102 to J2, J201 to J3, J202 to J4, J203 to J5, J204 to J6, Q101 to Q1, Q201 to Q2, Q202 to Q3, R101 to R1, R203 to R10, R204 to R11, R205 to R12, R102 to R2, R103 to R3, R104 to R4, R105 to R5, R106 to R6, R107 to R7, R201 to R8, R202 to R9, SW201 to SW1, SW202 to SW2, U101 to U1, U102 to U2, U202 to U5
Other:
- rule pad_to_mask_clearance: 0.1 -> 0.05

Commit message: Corrijo indicaciones de compañero
Parts:
- added G***: LOGO, tp_abbate:logo_unrn_B.Cu, F.Cu at (100.5, 82.0)
- J3: footprint U.FL:HRS_U.FL-R-SMT-1(10) -> tp_abbate:HRS_U.FL-R-SMT-1(10)
- turned C2 to 270 degrees
Connections:
- C2 pad 1: GND -> +5V
- C2 pad 2: +5V -> GND
Other:
- board text added: "20200626"
- board text added: "Diseñado en Argentina"
- board text added: "Wifi_LoRa_32 V1"

Commit message: Revisión Final - Entrega
Parts:
- added H1: MountingHole, tp_abbate:MountingHole_1.8mm_M3, F.Cu at (107.0, 80.8)
- added H2: MountingHole, tp_abbate:MountingHole_1.8mm_M3, F.Cu at (145.0, 87.8)
- added H3: MountingHole, tp_abbate:MountingHole_1.8mm_M3, F.Cu at (93.0, 118.2)
- added H4: MountingHole, tp_abbate:MountingHole_1.8mm_M3, F.Cu at (145.0, 111.2)
Routing:
- net +5V: track 111.0 -> 108.4 mm
- net /ESP32/CHIP_PU: track 90.8 -> 89.6 mm
